Commit message: added ros2_control for gazebo, 'yaml' files and updated launch files

File: description/robot.urdf.xacro (robot description, xacro)
@@ -1,5 +1,13 @@
 <?xml version="1.0"?>
 <robot xmlns:xacro="http://www.ros.org/wiki/xacro"  name="robot">
+    <xacro:arg name="use_ros2_control" default="true"/>
     <xacro:include filename="robot_core.xacro" />
-    <xacro:include filename="gazebo_control.xacro"/>
+    <xacro:if value="$(arg use_ros2_control)">
+        <!--ROS2 CONTROL SYSTEM-->
+        <xacro:include filename="ros2_control.xacro"/>
+    </xacro:if>
+    <xacro:unless value="$(arg use_ros2_control)">
+        <!-- GAZEBO CONTROL SYSTEM-->
+        <xacro:include filename="gazebo_control.xacro"/>
+    </xacro:unless>
 </robot>

File: description/robot_core.xacro (robot description, xacro)
@@ -60,5 +60,5 @@
         <collision>
             <geometry>
-                <cylinder radius="0.05" length="0.04"/>
+                <sphere radius="0.05"/>
             </geometry>
         </collision>
@@ -86,5 +86,5 @@
         <collision>
             <geometry>
-                <cylinder radius="0.05" length="0.04"/>
+                <sphere radius="0.05"/>
             </geometry>
         </collision>
